Commit message: gazebo no robot display

File: urdf/panda.urdf (robot description, URDF)
Before this commit: robot panda, 12 links, 11 joints
Links:
- link panda_hand: mass 0.73 -> None
- link panda_leftfinger: mass 0.015 -> None
- link panda_link0: mass 0.629769 -> None
- link panda_link1: mass 4.970684 -> None
- link panda_link2: mass 0.646926 -> None
- link panda_link3: mass 3.228604 -> None
- link panda_link4: mass 3.587895 -> None
- link panda_link5: mass 1.225946 -> None
- link panda_link6: mass 1.666555 -> None
- link panda_link7: mass 7.35522E-1 -> None
- link panda_rightfinger: mass 0.15 -> None

File: urdf/panda_gazebo.urdf.xacro (robot description, xacro)
@@ -54,5 +54,7 @@
   <!-- Include the base Panda URDF from moveit_resources -->
   <!-- ============================================= -->
-  <xacro:include filename="/home/ub22/ros2_ws/install/my_gazebo_learn/share/my_gazebo_learn/urdf/panda.urdf.xacro" />
+  <!--<xacro:include filename="/home/ub22/ros2_ws/src/my_gazebo_learn/urdf/panda.urdf.xacro" /> -->
+  <!-- <xacro:include filename="$(find moveit_resources_panda_moveit_config)/config/panda.urdf.xacro" />-->
+  <xacro:include filename="$(find my_gazebo_learn)/urdf/panda.urdf.xacro" />
   <!-- The moveit_resources_panda_description xacro macro call -->
   <!-- ============================================= -->
@@ -60,5 +62,4 @@
   <!-- ============================================= -->
   <!-- Gazebo ros2_control plugin for the arm -->
-<!--
   <gazebo>
     <plugin name="gazebo_ros2_control" filename="libgazebo_ros2_control.so">
@@ -68,40 +69,3 @@
     </plugin>
   </gazebo>
--->
-  <!-- ============================================= -->
-  <!-- ros2_control transmissions -->
-  <!-- ============================================= -->
-  <xacro:macro name="panda_transmission" params="joint_name">
-    <transmission name="trans_${joint_name}">
-      <type>transmission_interface/SimpleTransmission</type>
-      <joint name="${joint_name}">
-        <hardwareInterface>hardware_interface/EffortJointInterface</hardwareInterface>
-      </joint>
-      <actuator name="motor_${joint_name}">
-        <hardwareInterface>hardware_interface/EffortJointInterface</hardwareInterface>
-        <mechanicalReduction>1</mechanicalReduction>
-      </actuator>
-    </transmission>
-  </xacro:macro>
-  <xacro:panda_transmission joint_name="panda_joint1"/>
-  <xacro:panda_transmission joint_name="panda_joint2"/>
-  <xacro:panda_transmission joint_name="panda_joint3"/>
-  <xacro:panda_transmission joint_name="panda_joint4"/>
-  <xacro:panda_transmission joint_name="panda_joint5"/>
-  <xacro:panda_transmission joint_name="panda_joint6"/>
-  <xacro:panda_transmission joint_name="panda_joint7"/>
-  <xacro:macro name="panda_finger_transmission" params="joint_name">
-    <transmission name="trans_${joint_name}">
-      <type>transmission_interface/SimpleTransmission</type>
-      <joint name="${joint_name}">
-        <hardwareInterface>hardware_interface/EffortJointInterface</hardwareInterface>
-      </joint>
-      <actuator name="motor_${joint_name}">
-        <hardwareInterface>hardware_interface/EffortJointInterface</hardwareInterface>
-        <mechanicalReduction>1</mechanicalReduction>
-      </actuator>
-    </transmission>
-  </xacro:macro>
-  <xacro:panda_finger_transmission joint_name="panda_finger_joint1"/>
-  <xacro:panda_finger_transmission joint_name="panda_finger_joint2"/>
 </robot>
